Commit message: rto_description: rename content to reflect package name change

File: rto_description/urdf/components/robotino_body.urdf.xacro (robot description, xacro)
@@ -20,5 +20,5 @@
                 <origin xyz="0.01 0 0" rpy="0 0 ${M_PI/2}"/>
                 <geometry>
-                    <mesh filename="package://robotino_description/meshes/parts/robotino_base.dae"
+                    <mesh filename="package://rto_description/meshes/parts/robotino_base.dae"
                         scale="${M_SCALE} ${M_SCALE} ${M_SCALE}"/>
                 </geometry>

File: rto_description/urdf/components/robotino_parts.urdf.xacro (robot description, xacro)
@@ -16,5 +16,5 @@
                 <origin xyz="0 0 0" rpy="0 0 0"/>
                 <geometry>
-                    <mesh filename="package://robotino_description/meshes/parts/robotino_wheel.dae" scale="${M_SCALE} ${M_SCALE} ${M_SCALE}"/>
+                    <mesh filename="package://rto_description/meshes/parts/robotino_wheel.dae" scale="${M_SCALE} ${M_SCALE} ${M_SCALE}"/>
                 </geometry>
             </visual>
@@ -67,5 +67,5 @@
                 <origin xyz="0 0 0" rpy="0 0 0"/>
                 <geometry>
-                    <mesh filename="package://robotino_description/meshes/parts/angle_bracket_usb_hub.dae" scale="${M_SCALE} ${M_SCALE} ${M_SCALE}"/>
+                    <mesh filename="package://rto_description/meshes/parts/angle_bracket_usb_hub.dae" scale="${M_SCALE} ${M_SCALE} ${M_SCALE}"/>
                 </geometry>
             </visual>

File: rto_description/urdf/robots/robotino.urdf (robot description, URDF)
Before this commit: robot robotino, 6 links, 5 joints
Links:
- link anglebracketusb_link: geometry visual mesh filename=package://rto_description/meshes/parts/angle_bracket_usb_hu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 scale=0.01 0.01 0.01
- link base_link: geometry collision cylinder length=0.05 radius=0.18; visual mesh filename=package://rto_description/meshes/parts/robotino_base.dae scale=0.01 0.01 0.01
- link wheel0_link: geometry visual mesh filename=package://rto_description/meshes/parts/robotino_wheel.dae scale=0.01 0.01 0.01
- link wheel1_link: geometry visual mesh filename=package://rto_description/meshes/parts/robotino_wheel.dae scale=0.01 0.01 0.01
- link wheel2_link: geometry visual mesh filename=package://rto_description/meshes/parts/robotino_wheel.dae scale=0.01 0.01 0.01

File: rto_description/urdf/robots/robotino.urdf.xacro (robot description, xacro)
@@ -1,6 +1,6 @@
 <?xml version="1.0"?>
 <robot name="robotino" xmlns:xacro="http://wiki.ros.org/xacro">
-  <xacro:include filename="$(find robotino_description)/urdf/robotino_body.urdf.xacro"/>
-  <xacro:include filename="$(find robotino_description)/urdf/robotino_parts.urdf.xacro"/>
+  <xacro:include filename="$(find rto_description)/urdf/robotino_body.urdf.xacro"/>
+  <xacro:include filename="$(find rto_description)/urdf/robotino_parts.urdf.xacro"/>
   <xacro:robotino_body/>
 </robot>

File: rto_description/urdf/robots/robotino_description.urdf (robot description, URDF)
Before this commit: robot robotino, 6 links, 5 joints
Links:
- link anglebracketusb_link: geometry visual mesh filename=package://rto_description/meshes/parts/angle_bracket_usb_hu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 scale=0.01 0.01 0.01
- link base_link: geometry collision cylinder length=0.05 radius=0.18; visual mesh filename=package://rto_description/meshes/parts/robotino_base.dae scale=0.01 0.01 0.01
- link wheel0_link: geometry visual mesh filename=package://rto_description/meshes/parts/robotino_wheel.dae scale=0.01 0.01 0.01
- link wheel1_link: geometry visual mesh filename=package://rto_description/meshes/parts/robotino_wheel.dae scale=0.01 0.01 0.01
- link wheel2_link: geometry visual mesh filename=package://rto_description/meshes/parts/robotino_wheel.dae scale=0.01 0.01 0.01

File: rto_description/urdf/robots/robotino_description.urdf.xacro (robot description, xacro)
@@ -2,8 +2,8 @@
 <robot name="robotino" xmlns:xacro="http://wiki.ros.org/xacro">
    <!-- Instanciate and include the robotino_body -->
-  <xacro:include filename="$(find robotino_description)/urdf/components/robotino_body.urdf.xacro"/>
+  <xacro:include filename="$(find rto_description)/urdf/components/robotino_body.urdf.xacro"/>
   <xacro:robotino_body/>
    <!-- Instanciate and include the robotino_parts -->
-  <xacro:include filename="$(find robotino_description)/urdf/components/robotino_parts.urdf.xacro"/>
+  <xacro:include filename="$(find rto_description)/urdf/components/robotino_parts.urdf.xacro"/>
   <xacro:wheel name="wheel0" parent="base_link">
     <origin xyz="0.065 0.11 0.04" rpy="0 0 1.04719666667"/>
@@ -24,5 +24,5 @@
     <origin rpy="0 0 1.570795" xyz="0.008 0 0.137"/>
   </xacro:anglebracketusb>
-  <xacro:include filename="$(find robotino_description)/urdf/sensors/Sharp_IR_Sensor.urdf.xacro"/>
+  <xacro:include filename="$(find rto_description)/urdf/sensors/Sharp_IR_Sensor.urdf.xacro"/>
   <xacro:Ir_sensor name="ir1" parent="base_link">
     <origin rpy="0 0 0" xyz="0 -0.2264 0.0566" />

File: rto_description/urdf/sensors/Sharp_IR_Sensor.urdf.xacro (robot description, xacro)
@@ -15,5 +15,5 @@
         <origin xyz="0 0 0" rpy="0 0 0" />
         <geometry>
-          <mesh filename="package://robotino_description/meshes/sensors/Sharp_IR_Sensor_GP2Y0A41SK0F.dae" scale="${M_SCALE} ${M_SCALE} ${M_SCALE}"/>
+          <mesh filename="package://rto_description/meshes/sensors/Sharp_IR_Sensor_GP2Y0A41SK0F.dae" scale="${M_SCALE} ${M_SCALE} ${M_SCALE}"/>
         </geometry>
       </visual>

File: rto_description/urdf/sensors/asus_xtion_pro.urdf.xacro (robot description, xacro)
@@ -1,5 +1,5 @@
 <?xml version="1.0"?>
 <robot name="sensor_asus_xtion_pro" xmlns:xacro="http://ros.org/wiki/xacro">
-  <xacro:include filename="$(find robotino_description)/urdf/3dsensor_gazebo.urdf.xacro"/>
+  <xacro:include filename="$(find rto_description)/urdf/3dsensor_gazebo.urdf.xacro"/>
   <xacro:property name="M_SCALE" value="0.001"/>
   <xacro:property name="asus_xtion_pro_depth_rel_rgb_py" value="0.0270" />
@@ -51,5 +51,5 @@
         <origin xyz="-0.01 0 0" rpy="${-M_PI/2} -${M_PI} ${-M_PI/2}"/>
         <geometry>
-          <mesh filename="package://robotino_description/meshes/sensors/asus_xtion_pro_live.dae" scale="${M_SCALE} ${M_SCALE} ${M_SCALE}"/>
+          <mesh filename="package://rto_description/meshes/sensors/asus_xtion_pro_live.dae" scale="${M_SCALE} ${M_SCALE} ${M_SCALE}"/>
         </geometry>
       </visual>

File: rto_description/urdf/sensors/camera.urdf.xacro (robot description, xacro)
@@ -20,5 +20,5 @@
         <origin xyz="0 0 0" rpy="0 0 0" />
         <geometry>
-          <mesh filename="package://robotino_description/meshes/sensors/camera.dae" scale="${M_SCALE} ${M_SCALE} ${M_SCALE}"/>
+          <mesh filename="package://rto_description/meshes/sensors/camera.dae" scale="${M_SCALE} ${M_SCALE} ${M_SCALE}"/>
         </geometry>
       </visual>

File: rto_description/urdf/sensors/hokuyo.urdf.xacro (robot description, xacro)
@@ -23,5 +23,5 @@
         <geometry>
           <mesh
-filename="package://robotino_description/meshes/sensors/hokuyo.dae" scale="${M_SCALE} ${M_SCALE} ${M_SCALE}"/>
+filename="package://rto_description/meshes/sensors/hokuyo.dae" scale="${M_SCALE} ${M_SCALE} ${M_SCALE}"/>
         </geometry>
       </visual>

File: rto_description/urdf/sensors/kinect.urdf.xacro (robot description, xacro)
@@ -1,5 +1,5 @@
 <?xml version="1.0"?>
 <robot name="sensor_kinect" xmlns:xacro="http://ros.org/wiki/xacro">
-  <xacro:include filename="$(find robotino_description)/urdf/sensors/3dsensor_gazebo.urdf.xacro"/>
+  <xacro:include filename="$(find rto_description)/urdf/sensors/3dsensor_gazebo.urdf.xacro"/>
   <xacro:property name="KINECT_LENGTH" value="0.064"/>
   <xacro:property name="KINECT_WIDTH" value="0.121"/>
@@ -23,5 +23,5 @@
         <!-- <origin xyz="0 0 0" rpy="0 0 0" /> -->
         <geometry>
-          <mesh filename="package://robotino_description/meshes/sensors/kinect.dae"/>
+          <mesh filename="package://rto_description/meshes/sensors/kinect.dae"/>
           <!-- <box size="${KINECT_LENGTH} ${KINECT_WIDTH} ${KINECT_HEIGHT}"/> -->
         </geometry>
